Commit message: stable version

File: src/my_robot_description/urdf/my_wheelchair.urdf.xacro (robot description, xacro)
@@ -1,5 +1,5 @@
 <?xml version="1.0"?>
 <robot name="Wheelchair_urdf" xmlns:xacro="http://www.ros.org/wiki/xacro">
-    <!-- <xacro:include filename="common_properties.xacro" /> -->
+    <xacro:include filename="common_properties.xacro" />
     <xacro:include filename="wheelchair_base.xacro" />
     <xacro:include filename="wheelchair_base.ros2_control.xacro" />

File: src/my_robot_description/urdf/wheelchair_base.ros2_control.xacro (robot description, xacro)
@@ -3,26 +3,19 @@
     <ros2_control name="MobileBaseHardwareInterface" type="system">
         <hardware>
-            <plugin>mock_components/GenericSystem</plugin>
+            <plugin>gz_ros2_control/GazeboSimSystem</plugin>
+            <!-- <plugin>mock_components/GenericSystem</plugin> -->
             <param name="calculate_dynamics">true</param>
         </hardware>
+        <joint name="lf_1_joint">
+            <state_interface name="position" />
+        </joint>
+        <joint name="rf_1_joint">
+            <state_interface name="position" />
+        </joint>
         <joint name="lf_2_joint">
-            <command_interface name="velocity" />
             <state_interface name="position" />
-            <state_interface name="velocity" />
-        </joint>
-        <joint name="lf_1_joint">
-            <command_interface name="velocity" />
-            <state_interface name="position" />
-            <state_interface name="velocity" />
         </joint>
         <joint name="rf_2_joint">
-            <command_interface name="velocity" />
             <state_interface name="position" />
-            <state_interface name="velocity" />
-        </joint>
-        <joint name="rf_1_joint">
-            <command_interface name="velocity" />
-            <state_interface name="position" />
-            <state_interface name="velocity" />
         </joint>
         <joint name="rb_1_joint">

File: src/my_robot_description/urdf/wheelchair_base.xacro (robot description, xacro)
@@ -5,4 +5,13 @@
      For more information, please see http://wiki.ros.org/sw_urdf_exporter -->
 <robot name="Wheelchair_urdf" xmlns:xacro="http://www.ros.org/wiki/xacro">
+  <xacro:include filename="$(find my_robot_description)/urdf/wheelchair_gazebo.urdf.xacro" />
+  <xacro:property name="base_to_ground_z" value="0.7625" />
+  <link name="base_footprint" />
+  <joint name="base_footprint_joint" type="fixed">
+    <origin xyz="0 0 ${base_to_ground_z}" rpy="0 0 0" />
+    <parent link="base_footprint" />
+    <child link="base_link" />
+    <axis xyz="0 0 0" />
+  </joint>
   <link name="base_link">
     <inertial>
@@ -118,5 +127,5 @@
     </inertial>
     <visual>
-      <origin xyz="0 0 0" rpy="0 0 0" />
+      <origin xyz="0 0 0.0" rpy="0 0 0" />
       <geometry>
         <mesh filename="file://$(find my_robot_description)/meshes/lf_2.STL" />
@@ -127,5 +136,5 @@
     </visual>
     <collision>
-      <origin xyz="0 0 0" rpy="0 0 0" />
+      <origin xyz="0 0 0.0" rpy="0 0 0" />
       <geometry>
         <mesh filename="file://$(find my_robot_description)/meshes/lf_2.STL" />
@@ -134,5 +143,5 @@
   </link>
   <joint name="lf_2_joint" type="continuous">
-    <origin xyz="0.32552 0.38188 -0.5095" rpy="0 0 3.1416" />
+    <origin xyz="0.32552 0.38188 -0.5095" rpy="0 0 3.14159" />
     <parent link="base_link" />
     <child link="lf_2" />
@@ -146,5 +155,5 @@
     </inertial>
     <visual>
-      <origin xyz="0 0 0" rpy="0 0 0" />
+      <origin xyz="0 0 0.0" rpy="0 0 0" />
       <geometry>
         <mesh filename="file://$(find my_robot_description)/meshes/lf_1.STL" />
@@ -155,5 +164,5 @@
     </visual>
     <collision>
-      <origin xyz="0 0 0" rpy="0 0 0" />
+      <origin xyz="0 0 0.0" rpy="0 0 0" />
       <geometry>
         <mesh filename="file://$(find my_robot_description)/meshes/lf_1.STL" />
@@ -174,5 +183,5 @@
     </inertial>
     <visual>
-      <origin xyz="0 0 0" rpy="0 0 0" />
+      <origin xyz="0 0 0.0" rpy="0 0 0" />
       <geometry>
         <mesh filename="file://$(find my_robot_description)/meshes/rf_2.STL" />
@@ -183,5 +192,5 @@
     </visual>
     <collision>
-      <origin xyz="0 0 0" rpy="0 0 0" />
+      <origin xyz="0 0 0.0" rpy="0 0 0" />
       <geometry>
         <mesh filename="file://$(find my_robot_description)/meshes/rf_2.STL" />
@@ -202,5 +211,5 @@
     </inertial>
     <visual>
-      <origin xyz="0 0 0" rpy="0 0 0" />
+      <origin xyz="0 0 0.0" rpy="0 0 0" />
       <geometry>
         <mesh filename="file://$(find my_robot_description)/meshes/rf_1.STL" />
@@ -211,5 +220,5 @@
     </visual>
     <collision>
-      <origin xyz="0 0 0" rpy="0 0 0" />
+      <origin xyz="0 0 0.0" rpy="0 0 0" />
       <geometry>
         <mesh filename="file://$(find my_robot_description)/meshes/rf_1.STL" />
@@ -230,5 +239,5 @@
     </inertial>
     <visual>
-      <origin xyz="0 0 0" rpy="0 0 0" />
+      <origin xyz="0 0 0.0" rpy="0 0 0" />
       <geometry>
         <mesh filename="file://$(find my_robot_description)/meshes/rb_1.STL" />
@@ -239,5 +248,5 @@
     </visual>
     <collision>
-      <origin xyz="0 0 0" rpy="0 0 0" />
+      <origin xyz="0 0 0.0" rpy="0 0 0" />
       <geometry>
         <mesh filename="file://$(find my_robot_description)/meshes/rb_1.STL" />
@@ -253,10 +262,10 @@
   <link name="lb_1">
     <inertial>
-      <origin xyz="0 0 0" rpy="0 0 0" />
-      <mass value="0" />
-      <inertia ixx="0" ixy="0" ixz="0" iyy="0" iyz="0" izz="0" />
-    </inertial>
-    <visual>
-      <origin xyz="0 0 0" rpy="0 0 0" />
+      <origin xyz="2.9846E-09 1.1851E-09 0.060456" rpy="0 0 0" />
+      <mass value="6.8929" />
+      <inertia ixx="0.051089" ixy="-2.9975E-11" ixz="-1.9576E-10" iyy="0.051089" iyz="-4.6179E-11" izz="0.093148" />
+    </inertial>
+    <visual>
+      <origin xyz="0 0 0.0" rpy="0 0 0" />
       <geometry>
         <mesh filename="file://$(find my_robot_description)/meshes/lb_1.STL" />
@@ -267,5 +276,5 @@
     </visual>
     <collision>
-      <origin xyz="0 0 0" rpy="0 0 0" />
+      <origin xyz="0 0 0.0" rpy="0 0 0" />
       <geometry>
         <mesh filename="file://$(find my_robot_description)/meshes/lb_1.STL" />
@@ -279,3 +288,51 @@
     <axis xyz="0 0 1" />
   </joint>
+  <link name="imu_link">
+    <inertial>
+      <origin xyz="-0.00552433659106688 0.000168210391520346 0.000514000497342681" rpy="0 0 0" />
+      <mass value="0.000528415362211671" />
+      <inertia ixx="1.46176048428261E-08" ixy="1.40015117949421E-10" ixz="-1.99633872937403E-12" iyy="8.59662482954888E-09" iyz="7.52375112767959E-12" izz="2.30279421279312E-08" />
+    </inertial>
+    <visual>
+      <origin xyz="0 0 0" rpy="0 0 0" />
+      <geometry>
+        <mesh filename="file://$(find my_robot_description)/meshes/imu_link.STL" />
+      </geometry>
+      <material name="">
+        <color rgba="0.792156862745098 0.819607843137255 0.933333333333333 1" />
+      </material>
+    </visual>
+    <collision>
+      <origin xyz="0 0 0" rpy="0 0 0" />
+      <geometry>
+        <mesh filename="file://$(find my_robot_description)/meshes/imu_link.STL" />
+      </geometry>
+    </collision>
+  </link>
+  <joint name="imu_joint" type="fixed">
+    <origin xyz="0 0 ${base_to_ground_z}" rpy="0 0 0" />
+    <parent link="base_link"/>
+    <child link="imu_link"/>
+    <axis xyz="0 0 0" />
+  </joint>
+  <transmission name="lb_trans">
+    <type>transmission_interface/SimpleTransmission</type>
+    <joint name="lb_1_joint">
+      <hardwareInterface>hardware_interface/EffortJointInterface</hardwareInterface>
+    </joint>
+    <actuator name="lb_motor">
+      <hardwareInterface>hardware_interface/EffortJointInterface</hardwareInterface>
+      <mechanicalReduction>1</mechanicalReduction>
+    </actuator>
+  </transmission>
+  <transmission name="rb_trans">
+    <type>transmission_interface/SimpleTransmission</type>
+    <joint name="rb_1_joint">
+      <hardwareInterface>hardware_interface/EffortJointInterface</hardwareInterface>
+    </joint>
+    <actuator name="rb_motor">
+      <hardwareInterface>hardware_interface/EffortJointInterface</hardwareInterface>
+      <mechanicalReduction>1</mechanicalReduction>
+    </actuator>
+  </transmission>
 </robot>
