Commit message: Launching wheelchair in gazebo

File: src/my_robot_description/urdf/wheelchair_base.ros2_control.xacro (robot description, xacro)
@@ -3,6 +3,7 @@
     <ros2_control name="MobileBaseHardwareInterface" type="system">
         <hardware>
-            <plugin>mock_components/GenericSystem</plugin>
-            <param name="calculate_dynamics">true</param>
+            <plugin>gz_ros2_control/GazeboSimSystem</plugin>
+            <!-- <plugin>mock_components/GenericSystem</plugin> -->
+            <!-- <param name="calculate_dynamics">true</param> -->
         </hardware>
         <joint name="lf_2_joint">
@@ -36,4 +37,16 @@
             <state_interface name="velocity" />
         </joint>
+        <!-- <sensor name="imu">
+            <state_interface name="orientation.x"/>
+            <state_interface name="orientation.y"/>
+            <state_interface name="orientation.z"/>
+            <state_interface name="orientation.w"/>
+            <state_interface name="angular_velocity.x"/>
+            <state_interface name="angular_velocity.y"/>
+            <state_interface name="angular_velocity.z"/>
+            <state_interface name="linear_acceleration.x"/>
+            <state_interface name="linear_acceleration.y"/>
+            <state_interface name="linear_acceleration.z"/>
+        </sensor> -->
     </ros2_control>
 </robot>

File: src/my_robot_description/urdf/wheelchair_base.xacro (robot description, xacro)
@@ -254,6 +254,6 @@
     <inertial>
       <origin xyz="0 0 0" rpy="0 0 0" />
-      <mass value="0" />
-      <inertia ixx="0" ixy="0" ixz="0" iyy="0" iyz="0" izz="0" />
+      <mass value="6.8929" />
+      <inertia ixx="0.051089" ixy="-2.9975E-11" ixz="-1.9576E-10" iyy="0.051089" iyz="-4.6179E-11" izz="0.093148" />
     </inertial>
     <visual>
@@ -279,3 +279,31 @@
     <axis xyz="0 0 1" />
   </joint>
+  <link name="imu_link">
+    <inertial>
+      <mass value="0.01"/>
+      <origin xyz="0 0 0" rpy="0 0 0"/>
+      <inertia ixx="0.0001" iyy="0.0001" izz="0.0001" ixy="0" ixz="0" iyz="0"/>
+    </inertial>
+    <visual>
+      <origin xyz="0 0 0" rpy="0 0 0" />
+      <geometry>
+        <mesh filename="file://$(find my_robot_description)/meshes/imu_link.STL" />
+      </geometry>
+      <material name="">
+        <color rgba="0.792156862745098 0.819607843137255 0.933333333333333 1" />
+      </material>
+      <collision>
+      <origin xyz="0 0 0" rpy="0 0 0" />
+      <geometry>
+        <mesh filename="file://$(find my_robot_description)/meshes/imu_link.STL" />
+      </geometry>
+    </collision>
+    </visual>
+  </link>
+  <joint name="imu_joint" type="fixed">
+    <origin xyz="0 0 -0.0698986241758014" rpy="0 0 0" />
+    <parent link="base_link"/>
+    <child link="imu_link"/>
+    <axis xyz="0 0 0" />
+  </joint>
 </robot>

Commit message: wheelchair simulated in gazebo

File: src/my_robot_description/urdf/wheelchair_base.ros2_control.xacro (robot description, xacro)
@@ -5,5 +5,5 @@
             <plugin>gz_ros2_control/GazeboSimSystem</plugin>
             <!-- <plugin>mock_components/GenericSystem</plugin> -->
-            <!-- <param name="calculate_dynamics">true</param> -->
+            <param name="calculate_dynamics">true</param>
         </hardware>
         <joint name="lf_2_joint">

File: src/my_robot_description/urdf/wheelchair_base.xacro (robot description, xacro)
@@ -5,4 +5,5 @@
      For more information, please see http://wiki.ros.org/sw_urdf_exporter -->
 <robot name="Wheelchair_urdf" xmlns:xacro="http://www.ros.org/wiki/xacro">
+  <xacro:include filename="$(find my_robot_description)/urdf/wheelchair_gazebo.urdf.xacro" />
   <link name="base_link">
     <inertial>
@@ -281,7 +282,9 @@
   <link name="imu_link">
     <inertial>
-      <mass value="0.01"/>
-      <origin xyz="0 0 0" rpy="0 0 0"/>
-      <inertia ixx="0.0001" iyy="0.0001" izz="0.0001" ixy="0" ixz="0" iyz="0"/>
+      <origin xyz="-0.00552433659106688 0.000168210391520346 0.000514000497342681" rpy="0 0 0" />
+      <mass value="0.000528415362211671" />
+      <inertia ixx="1.46176048428261E-08" ixy="1.40015117949421E-10" ixz="-1.99633872937403E-12"
+               iyy="8.59662482954888E-09" iyz="7.52375112767959E-12"
+               izz="2.30279421279312E-08" />
     </inertial>
     <visual>
@@ -293,5 +296,6 @@
         <color rgba="0.792156862745098 0.819607843137255 0.933333333333333 1" />
       </material>
-      <collision>
+    </visual>
+    <collision>
       <origin xyz="0 0 0" rpy="0 0 0" />
       <geometry>
@@ -299,8 +303,7 @@
       </geometry>
     </collision>
-    </visual>
   </link>
   <joint name="imu_joint" type="fixed">
-    <origin xyz="0 0 -0.0698986241758014" rpy="0 0 0" />
+    <origin xyz="0 0 -0.07" rpy="0 0 0" />
     <parent link="base_link"/>
     <child link="imu_link"/>

Commit message: Wheelchair Lidar simulated

File: src/my_robot_description/urdf/wheelchair_base.ros2_control.xacro (robot description, xacro)
@@ -7,9 +7,9 @@
             <param name="calculate_dynamics">true</param>
         </hardware>
-        <joint name="lf_2_joint">
+        <!-- <joint name="lf_2_joint">
             <command_interface name="velocity" />
             <state_interface name="position" />
             <state_interface name="velocity" />
-        </joint>
+        </joint> -->
         <joint name="lf_1_joint">
             <command_interface name="velocity" />
@@ -17,9 +17,9 @@
             <state_interface name="velocity" />
         </joint>
-        <joint name="rf_2_joint">
+        <!-- <joint name="rf_2_joint">
             <command_interface name="velocity" />
             <state_interface name="position" />
             <state_interface name="velocity" />
-        </joint>
+        </joint> -->
         <joint name="rf_1_joint">
             <command_interface name="velocity" />

File: src/my_robot_description/urdf/wheelchair_base.xacro (robot description, xacro)
@@ -134,6 +134,6 @@
     </collision>
   </link>
-  <joint name="lf_2_joint" type="continuous">
-    <origin xyz="0.32552 0.38188 -0.5095" rpy="0 0 3.1416" />
+  <joint name="lf_2_joint" type="fixed">
+    <origin xyz="0.32552 0.38188 -0.5095" rpy="0 0 0" />
     <parent link="base_link" />
     <child link="lf_2" />
@@ -158,5 +158,5 @@
       <origin xyz="0 0 0" rpy="0 0 0" />
       <geometry>
-        <mesh filename="file://$(find my_robot_description)/meshes/lf_1.STL" />
+        <sphere radius="0.14"/>
       </geometry>
     </collision>
@@ -190,5 +190,5 @@
     </collision>
   </link>
-  <joint name="rf_2_joint" type="continuous">
+  <joint name="rf_2_joint" type="fixed">
     <origin xyz="0.32552 -0.38188 -0.5095" rpy="0 0 0" />
     <parent link="base_link" />
@@ -214,5 +214,5 @@
       <origin xyz="0 0 0" rpy="0 0 0" />
       <geometry>
-        <mesh filename="file://$(find my_robot_description)/meshes/rf_1.STL" />
+        <sphere radius="0.14"/>
       </geometry>
     </collision>
@@ -242,5 +242,5 @@
       <origin xyz="0 0 0" rpy="0 0 0" />
       <geometry>
-        <mesh filename="file://$(find my_robot_description)/meshes/rb_1.STL" />
+        <sphere radius="0.14"/>
       </geometry>
     </collision>
@@ -270,5 +270,5 @@
       <origin xyz="0 0 0" rpy="0 0 0" />
       <geometry>
-        <mesh filename="file://$(find my_robot_description)/meshes/lb_1.STL" />
+        <sphere radius="0.14"/>
       </geometry>
     </collision>

File: src/my_robot_description/urdf/wheelchair_gazebo.urdf.xacro (robot description, xacro)
@@ -40,4 +40,7 @@
         </plugin>
         <plugin filename="gz-sim-imu-system" name="gz::sim::systems::Imu"/>
+        <plugin filename="gz-sim-sensors-system" name="gz::sim::systems::Sensors">
+            <render_engine>ogre2</render_engine>
+        </plugin>
     </gazebo>
     <!-- IMU -->
@@ -92,3 +95,36 @@
         </sensor>
     </gazebo>
+    <!--Lidar-->
+    <gazebo reference='lidar_r'>
+        <sensor name='laser' type='gpu_lidar'>
+            <visualize>true</visualize>
+            <pose relative_to='lidar_r'>0 0 0 0 0 0</pose>
+            <update_rate>10</update_rate>
+            <gz_frame_id>lidar_r</gz_frame_id>
+            <topic>lidar</topic>
+            <ray>
+                <scan>
+                    <horizontal>
+                        <samples>640</samples>
+                        <resolution>1</resolution>
+                        <min_angle>-1.396263</min_angle>
+                        <max_angle>1.396263</max_angle>
+                    </horizontal>
+                    <vertical>
+                        <samples>1</samples>
+                        <resolution>0.01</resolution>
+                        <min_angle>0</min_angle>
+                        <max_angle>0</max_angle>
+                    </vertical>
+                </scan>
+                <range>
+                    <min>0.08</min>
+                    <max>10.0</max>
+                    <resolution>0.01</resolution>
+                </range>
+            </ray>
+            <always_on>1</always_on>
+            <visualize>true</visualize>
+        </sensor>
+    </gazebo>
 </robot>

Commit message: fixed motion

File: src/my_robot_description/urdf/wheelchair_base.ros2_control.xacro (robot description, xacro)
@@ -5,5 +5,5 @@
             <plugin>gz_ros2_control/GazeboSimSystem</plugin>
             <!-- <plugin>mock_components/GenericSystem</plugin> -->
-            <!-- <param name="calculate_dynamics">true</param> -->
+            <param name="calculate_dynamics">true</param>
         </hardware>
         <!-- <joint name="lf_2_joint">

File: src/my_robot_description/urdf/wheelchair_base.xacro (robot description, xacro)
@@ -135,5 +135,5 @@
   </link>
   <joint name="lf_2_joint" type="fixed">
-    <origin xyz="0.32552 0.38188 -0.5095" rpy="0 0 0" />
+    <origin xyz="0.32552 0.38188 -0.5095" rpy="0 0 3.14159" />
     <parent link="base_link" />
     <child link="lf_2" />

Commit message: syncing updates

File: src/my_robot_description/urdf/wheelchair_base.ros2_control.xacro (robot description, xacro)
@@ -1,9 +1,15 @@
 <?xml version="1.0"?>
 <robot xmlns:xacro="http://www.ros.org/wiki/xacro">
+    <xacro:arg name="use_mock_hardware" default="false"/>
     <ros2_control name="MobileBaseHardwareInterface" type="system">
         <hardware>
-            <plugin>gz_ros2_control/GazeboSimSystem</plugin>
-            <!-- <plugin>mock_components/GenericSystem</plugin> -->
-            <param name="calculate_dynamics">true</param>
+            <xacro:if value="$(arg use_mock_hardware)">
+                <plugin>mock_components/GenericSystem</plugin>
+                <param name="calculate_dynamics">true</param>
+            </xacro:if>
+            <xacro:unless value="$(arg use_mock_hardware)">
+                <plugin>gz_ros2_control/GazeboSimSystem</plugin>
+                <param name="calculate_dynamics">true</param>
+            </xacro:unless>
         </hardware>
         <joint name="lf_1_joint">

File: src/my_robot_description/urdf/wheelchair_base.xacro (robot description, xacro)
@@ -23,14 +23,14 @@
       <origin xyz="0 0 0" rpy="0 0 0" />
       <geometry>
-        <mesh filename="file://$(find my_robot_description)/meshes/wheelchair_meshes/base_link.STL" />
-      </geometry>
-      <material name="">
-        <color rgba="0.62745 0.62745 0.62745 1" />
-      </material>
-    </visual>
-    <collision>
-      <origin xyz="0 0 0" rpy="0 0 0" />
-      <geometry>
-        <mesh filename="file://$(find my_robot_description)/meshes/wheelchair_meshes/base_link.STL" />
+        <mesh filename="package://my_robot_description/meshes/wheelchair_meshes/base_link.STL" />
+      </geometry>
+      <material name="">
+        <color rgba="0.62745 0.62745 0.62745 1" />
+      </material>
+    </visual>
+    <collision>
+      <origin xyz="0 0 0" rpy="0 0 0" />
+      <geometry>
+        <mesh filename="package://my_robot_description/meshes/wheelchair_meshes/base_link.STL" />
       </geometry>
     </collision>
@@ -45,5 +45,5 @@
       <origin xyz="0 0 0" rpy="0 0 0" />
       <geometry>
-        <mesh filename="file://$(find my_robot_description)/meshes/wheelchair_meshes/lidar_r.STL" />
+        <mesh filename="package://my_robot_description/meshes/wheelchair_meshes/lidar_r.STL" />
       </geometry>
       <material name="">
@@ -54,5 +54,5 @@
       <origin xyz="0 0 0" rpy="0 0 0" />
       <geometry>
-        <mesh filename="file://$(find my_robot_description)/meshes/wheelchair_meshes/lidar_r.STL" />
+        <mesh filename="package://my_robot_description/meshes/wheelchair_meshes/lidar_r.STL" />
       </geometry>
     </collision>
@@ -73,5 +73,5 @@
       <origin xyz="0 0 0" rpy="0 0 0" />
       <geometry>
-        <mesh filename="file://$(find my_robot_description)/meshes/wheelchair_meshes/lidar_l.STL" />
+        <mesh filename="package://my_robot_description/meshes/wheelchair_meshes/lidar_l.STL" />
       </geometry>
       <material name="">
@@ -82,5 +82,5 @@
       <origin xyz="0 0 0" rpy="0 0 0" />
       <geometry>
-        <mesh filename="file://$(find my_robot_description)/meshes/wheelchair_meshes/lidar_l.STL" />
+        <mesh filename="package://my_robot_description/meshes/wheelchair_meshes/lidar_l.STL" />
       </geometry>
     </collision>
@@ -101,5 +101,5 @@
       <origin xyz="0 0 0" rpy="0 0 0" />
       <geometry>
-        <mesh filename="file://$(find my_robot_description)/meshes/wheelchair_meshes/lidar_t.STL" />
+        <mesh filename="package://my_robot_description/meshes/wheelchair_meshes/lidar_t.STL" />
       </geometry>
       <material name="">
@@ -110,5 +110,5 @@
       <origin xyz="0 0 0" rpy="0 0 0" />
       <geometry>
-        <mesh filename="file://$(find my_robot_description)/meshes/wheelchair_meshes/lidar_t.STL" />
+        <mesh filename="package://my_robot_description/meshes/wheelchair_meshes/lidar_t.STL" />
       </geometry>
     </collision>
@@ -129,14 +129,14 @@
       <origin xyz="0 0 0.0" rpy="0 0 0" />
       <geometry>
-        <mesh filename="file://$(find my_robot_description)/meshes/wheelchair_meshes/lf_2.STL" />
-      </geometry>
-      <material name="">
-        <color rgba="0.62745 0.62745 0.62745 1" />
-      </material>
-    </visual>
-    <collision>
-      <origin xyz="0 0 0.0" rpy="0 0 0" />
-      <geometry>
-        <mesh filename="file://$(find my_robot_description)/meshes/wheelchair_meshes/lf_2.STL" />
+        <mesh filename="package://my_robot_description/meshes/wheelchair_meshes/lf_2.STL" />
+      </geometry>
+      <material name="">
+        <color rgba="0.62745 0.62745 0.62745 1" />
+      </material>
+    </visual>
+    <collision>
+      <origin xyz="0 0 0.0" rpy="0 0 0" />
+      <geometry>
+        <mesh filename="package://my_robot_description/meshes/wheelchair_meshes/lf_2.STL" />
       </geometry>
     </collision>
@@ -157,14 +157,14 @@
       <origin xyz="0 0 0.0" rpy="0 0 0" />
       <geometry>
-        <mesh filename="file://$(find my_robot_description)/meshes/wheelchair_meshes/lf_1.STL" />
-      </geometry>
-      <material name="">
-        <color rgba="0.62745 0.62745 0.62745 1" />
-      </material>
-    </visual>
-    <collision>
-      <origin xyz="0 0 0.0" rpy="0 0 0" />
-      <geometry>
-        <mesh filename="file://$(find my_robot_description)/meshes/wheelchair_meshes/lf_1.STL" />
+        <mesh filename="package://my_robot_description/meshes/wheelchair_meshes/lf_1.STL" />
+      </geometry>
+      <material name="">
+        <color rgba="0.62745 0.62745 0.62745 1" />
+      </material>
+    </visual>
+    <collision>
+      <origin xyz="0 0 0.0" rpy="0 0 0" />
+      <geometry>
+        <mesh filename="package://my_robot_description/meshes/wheelchair_meshes/lf_1.STL" />
       </geometry>
     </collision>
@@ -185,14 +185,14 @@
       <origin xyz="0 0 0.0" rpy="0 0 0" />
       <geometry>
-        <mesh filename="file://$(find my_robot_description)/meshes/wheelchair_meshes/rf_2.STL" />
-      </geometry>
-      <material name="">
-        <color rgba="0.62745 0.62745 0.62745 1" />
-      </material>
-    </visual>
-    <collision>
-      <origin xyz="0 0 0.0" rpy="0 0 0" />
-      <geometry>
-        <mesh filename="file://$(find my_robot_description)/meshes/wheelchair_meshes/rf_2.STL" />
+        <mesh filename="package://my_robot_description/meshes/wheelchair_meshes/rf_2.STL" />
+      </geometry>
+      <material name="">
+        <color rgba="0.62745 0.62745 0.62745 1" />
+      </material>
+    </visual>
+    <collision>
+      <origin xyz="0 0 0.0" rpy="0 0 0" />
+      <geometry>
+        <mesh filename="package://my_robot_description/meshes/wheelchair_meshes/rf_2.STL" />
       </geometry>
     </collision>
@@ -213,14 +213,14 @@
       <origin xyz="0 0 0.0" rpy="0 0 0" />
       <geometry>
-        <mesh filename="file://$(find my_robot_description)/meshes/wheelchair_meshes/rf_1.STL" />
-      </geometry>
-      <material name="">
-        <color rgba="0.62745 0.62745 0.62745 1" />
-      </material>
-    </visual>
-    <collision>
-      <origin xyz="0 0 0.0" rpy="0 0 0" />
-      <geometry>
-        <mesh filename="file://$(find my_robot_description)/meshes/wheelchair_meshes/rf_1.STL" />
+        <mesh filename="package://my_robot_description/meshes/wheelchair_meshes/rf_1.STL" />
+      </geometry>
+      <material name="">
+        <color rgba="0.62745 0.62745 0.62745 1" />
+      </material>
+    </visual>
+    <collision>
+      <origin xyz="0 0 0.0" rpy="0 0 0" />
+      <geometry>
+        <mesh filename="package://my_robot_description/meshes/wheelchair_meshes/rf_1.STL" />
       </geometry>
     </collision>
@@ -241,14 +241,14 @@
       <origin xyz="0 0 0.0" rpy="0 0 0" />
       <geometry>
-        <mesh filename="file://$(find my_robot_description)/meshes/wheelchair_meshes/rb_1.STL" />
-      </geometry>
-      <material name="">
-        <color rgba="0.62745 0.62745 0.62745 1" />
-      </material>
-    </visual>
-    <collision>
-      <origin xyz="0 0 0.0" rpy="0 0 0" />
-      <geometry>
-        <mesh filename="file://$(find my_robot_description)/meshes/wheelchair_meshes/rb_1.STL" />
+        <mesh filename="package://my_robot_description/meshes/wheelchair_meshes/rb_1.STL" />
+      </geometry>
+      <material name="">
+        <color rgba="0.62745 0.62745 0.62745 1" />
+      </material>
+    </visual>
+    <collision>
+      <origin xyz="0 0 0.0" rpy="0 0 0" />
+      <geometry>
+        <mesh filename="package://my_robot_description/meshes/wheelchair_meshes/rb_1.STL" />
       </geometry>
     </collision>
@@ -269,5 +269,5 @@
       <origin xyz="0 0 0.0" rpy="0 0 0" />
       <geometry>
-        <mesh filename="file://$(find my_robot_description)/meshes/wheelchair_meshes/lb_1.STL" />
+        <mesh filename="package://my_robot_description/meshes/wheelchair_meshes/lb_1.STL" />
       </geometry>
       <material name="">
@@ -278,5 +278,5 @@
       <origin xyz="0 0 0.0" rpy="0 0 0" />
       <geometry>
-        <mesh filename="file://$(find my_robot_description)/meshes/wheelchair_meshes/lb_1.STL" />
+        <mesh filename="package://my_robot_description/meshes/wheelchair_meshes/lb_1.STL" />
       </geometry>
     </collision>
@@ -297,5 +297,5 @@
       <origin xyz="0 0 0" rpy="0 0 0" />
       <geometry>
-        <mesh filename="file://$(find my_robot_description)/meshes/wheelchair_meshes/imu_link.STL" />
+        <mesh filename="package://my_robot_description/meshes/wheelchair_meshes/imu_link.STL" />
       </geometry>
       <material name="">
@@ -306,5 +306,5 @@
       <origin xyz="0 0 0" rpy="0 0 0" />
       <geometry>
-        <mesh filename="file://$(find my_robot_description)/meshes/wheelchair_meshes/imu_link.STL" />
+        <mesh filename="package://my_robot_description/meshes/wheelchair_meshes/imu_link.STL" />
       </geometry>
     </collision>
