Commit message: Updated Arm

File: src/my_robot_description/urdf/arm_moveo_urdf.urdf (robot description, URDF)
Before this commit: robot my_robot_description, 15 links, 14 joints
Links:
- link Gripper_Idol_Gear: geometry collision mesh filename=file://$(find my_robot_description)/meshes/arm_meshes/Gripp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; visual mesh filename=file://$(find my_robot_description)/meshes/arm_meshes/Gripp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
- link Gripper_Servo_Gear: geometry collision mesh filename=file://$(find my_robot_description)/meshes/arm_meshes/Gripp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; visual mesh filename=file://$(find my_robot_description)/meshes/arm_meshes/Gripp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
- link Pivot_Arm_Gripper_Idol: geometry collision mesh filename=file://$(find my_robot_description)/meshes/arm_meshes/Pivot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; visual mesh filename=file://$(find my_robot_description)/meshes/arm_meshes/Pivot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
- link Pivot_Arm_Gripper_Servo: geometry collision mesh filename=file://$(find my_robot_description)/meshes/arm_meshes/Pivot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; visual mesh filename=file://$(find my_robot_description)/meshes/arm_meshes/Pivot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
- link Tip_Gripper_Idol: geometry collision mesh filename=file://$(find my_robot_description)/meshes/arm_meshes/Tip_G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; visual mesh filename=file://$(find my_robot_description)/meshes/arm_meshes/Tip_G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
- link Tip_Gripper_Servo: geometry collision mesh filename=file://$(find my_robot_description)/meshes/arm_meshes/Tip_G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; visual mesh filename=file://$(find my_robot_description)/meshes/arm_meshes/Tip_G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
- link arm_link: geometry collision mesh filename=file://$(find my_robot_description)/meshes/arm_meshes/Link_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; visual mesh filename=file://$(find my_robot_description)/meshes/arm_meshes/Link_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
- link base_link: geometry collision mesh filename=file://$(find my_robot_description)/meshes/arm_meshes/base_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; visual mesh filename=file://$(find my_robot_description)/meshes/arm_meshes/base_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
- link elbow_link: geometry collision mesh filename=file://$(find my_robot_description)/meshes/arm_meshes/Link_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; visual mesh filename=file://$(find my_robot_description)/meshes/arm_meshes/Link_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
- link forearm_link: geometry collision mesh filename=file://$(find my_robot_description)/meshes/arm_meshes/Link_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; visual mesh filename=file://$(find my_robot_description)/meshes/arm_meshes/Link_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
- link shoulder_link: geometry collision mesh filename=file://$(find my_robot_description)/meshes/arm_meshes/Link_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; visual mesh filename=file://$(find my_robot_description)/meshes/arm_meshes/Link_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
- link wrist_link: geometry collision mesh filename=file://$(find my_robot_description)/meshes/arm_meshes/Link_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; visual mesh filename=file://$(find my_robot_description)/meshes/arm_meshes/Link_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

File: src/my_robot_description/urdf/arm_urdf.xacro (robot description, xacro)
@@ -4,9 +4,9 @@
   <xacro:arg name="use_sim" default="false"/>
   <!-- Include other XACRO/URDF files -->
-  <xacro:include filename="$(find my_robot_description)/urdf/my_robot_description.ros2_control.xacro"/>
-  <xacro:include filename="$(find my_robot_description)/urdf/moveo_urdf.urdf"/>
+  <xacro:include filename="$(find my_robot_description)/urdf/arm_description.ros2_control.xacro"/>
+  <xacro:include filename="$(find my_robot_description)/urdf/arm_moveo_urdf.urdf"/>
   <gazebo>
     <plugin filename="gz_ros2_control-system" name="gz_ros2_control::GazeboSimROS2ControlPlugin">
-      <parameters>$(find my_robot_bringup)/config/ros2_controllers.yaml</parameters>
+      <parameters>$(find my_robot_bringup)/config/arm_controllers.yaml</parameters>
     </plugin>
   </gazebo>

File: src/my_robot_description/urdf/wheelchair_base.xacro (robot description, xacro)
@@ -23,14 +23,14 @@
       <origin xyz="0 0 0" rpy="0 0 0" />
       <geometry>
-        <mesh filename="file://$(find my_robot_description)/meshes/base_link.STL" />
-      </geometry>
-      <material name="">
-        <color rgba="0.62745 0.62745 0.62745 1" />
-      </material>
-    </visual>
-    <collision>
-      <origin xyz="0 0 0" rpy="0 0 0" />
-      <geometry>
-        <mesh filename="file://$(find my_robot_description)/meshes/base_link.STL" />
+        <mesh filename="file://$(find my_robot_description)/meshes/wheelchair_meshes/base_link.STL" />
+      </geometry>
+      <material name="">
+        <color rgba="0.62745 0.62745 0.62745 1" />
+      </material>
+    </visual>
+    <collision>
+      <origin xyz="0 0 0" rpy="0 0 0" />
+      <geometry>
+        <mesh filename="file://$(find my_robot_description)/meshes/wheelchair_meshes/base_link.STL" />
       </geometry>
     </collision>
@@ -45,5 +45,5 @@
       <origin xyz="0 0 0" rpy="0 0 0" />
       <geometry>
-        <mesh filename="file://$(find my_robot_description)/meshes/lidar_r.STL" />
+        <mesh filename="file://$(find my_robot_description)/meshes/wheelchair_meshes/lidar_r.STL" />
       </geometry>
       <material name="">
@@ -54,5 +54,5 @@
       <origin xyz="0 0 0" rpy="0 0 0" />
       <geometry>
-        <mesh filename="file://$(find my_robot_description)/meshes/lidar_r.STL" />
+        <mesh filename="file://$(find my_robot_description)/meshes/wheelchair_meshes/lidar_r.STL" />
       </geometry>
     </collision>
@@ -73,5 +73,5 @@
       <origin xyz="0 0 0" rpy="0 0 0" />
       <geometry>
-        <mesh filename="file://$(find my_robot_description)/meshes/lidar_l.STL" />
+        <mesh filename="file://$(find my_robot_description)/meshes/wheelchair_meshes/lidar_l.STL" />
       </geometry>
       <material name="">
@@ -82,5 +82,5 @@
       <origin xyz="0 0 0" rpy="0 0 0" />
       <geometry>
-        <mesh filename="file://$(find my_robot_description)/meshes/lidar_l.STL" />
+        <mesh filename="file://$(find my_robot_description)/meshes/wheelchair_meshes/lidar_l.STL" />
       </geometry>
     </collision>
@@ -101,5 +101,5 @@
       <origin xyz="0 0 0" rpy="0 0 0" />
       <geometry>
-        <mesh filename="file://$(find my_robot_description)/meshes/lidar_t.STL" />
+        <mesh filename="file://$(find my_robot_description)/meshes/wheelchair_meshes/lidar_t.STL" />
       </geometry>
       <material name="">
@@ -110,5 +110,5 @@
       <origin xyz="0 0 0" rpy="0 0 0" />
       <geometry>
-        <mesh filename="file://$(find my_robot_description)/meshes/lidar_t.STL" />
+        <mesh filename="file://$(find my_robot_description)/meshes/wheelchair_meshes/lidar_t.STL" />
       </geometry>
     </collision>
@@ -129,14 +129,14 @@
       <origin xyz="0 0 0.0" rpy="0 0 0" />
       <geometry>
-        <mesh filename="file://$(find my_robot_description)/meshes/lf_2.STL" />
-      </geometry>
-      <material name="">
-        <color rgba="0.62745 0.62745 0.62745 1" />
-      </material>
-    </visual>
-    <collision>
-      <origin xyz="0 0 0.0" rpy="0 0 0" />
-      <geometry>
-        <mesh filename="file://$(find my_robot_description)/meshes/lf_2.STL" />
+        <mesh filename="file://$(find my_robot_description)/meshes/wheelchair_meshes/lf_2.STL" />
+      </geometry>
+      <material name="">
+        <color rgba="0.62745 0.62745 0.62745 1" />
+      </material>
+    </visual>
+    <collision>
+      <origin xyz="0 0 0.0" rpy="0 0 0" />
+      <geometry>
+        <mesh filename="file://$(find my_robot_description)/meshes/wheelchair_meshes/lf_2.STL" />
       </geometry>
     </collision>
@@ -157,14 +157,14 @@
       <origin xyz="0 0 0.0" rpy="0 0 0" />
       <geometry>
-        <mesh filename="file://$(find my_robot_description)/meshes/lf_1.STL" />
-      </geometry>
-      <material name="">
-        <color rgba="0.62745 0.62745 0.62745 1" />
-      </material>
-    </visual>
-    <collision>
-      <origin xyz="0 0 0.0" rpy="0 0 0" />
-      <geometry>
-        <mesh filename="file://$(find my_robot_description)/meshes/lf_1.STL" />
+        <mesh filename="file://$(find my_robot_description)/meshes/wheelchair_meshes/lf_1.STL" />
+      </geometry>
+      <material name="">
+        <color rgba="0.62745 0.62745 0.62745 1" />
+      </material>
+    </visual>
+    <collision>
+      <origin xyz="0 0 0.0" rpy="0 0 0" />
+      <geometry>
+        <mesh filename="file://$(find my_robot_description)/meshes/wheelchair_meshes/lf_1.STL" />
       </geometry>
     </collision>
@@ -185,14 +185,14 @@
       <origin xyz="0 0 0.0" rpy="0 0 0" />
       <geometry>
-        <mesh filename="file://$(find my_robot_description)/meshes/rf_2.STL" />
-      </geometry>
-      <material name="">
-        <color rgba="0.62745 0.62745 0.62745 1" />
-      </material>
-    </visual>
-    <collision>
-      <origin xyz="0 0 0.0" rpy="0 0 0" />
-      <geometry>
-        <mesh filename="file://$(find my_robot_description)/meshes/rf_2.STL" />
+        <mesh filename="file://$(find my_robot_description)/meshes/wheelchair_meshes/rf_2.STL" />
+      </geometry>
+      <material name="">
+        <color rgba="0.62745 0.62745 0.62745 1" />
+      </material>
+    </visual>
+    <collision>
+      <origin xyz="0 0 0.0" rpy="0 0 0" />
+      <geometry>
+        <mesh filename="file://$(find my_robot_description)/meshes/wheelchair_meshes/rf_2.STL" />
       </geometry>
     </collision>
@@ -213,14 +213,14 @@
       <origin xyz="0 0 0.0" rpy="0 0 0" />
       <geometry>
-        <mesh filename="file://$(find my_robot_description)/meshes/rf_1.STL" />
-      </geometry>
-      <material name="">
-        <color rgba="0.62745 0.62745 0.62745 1" />
-      </material>
-    </visual>
-    <collision>
-      <origin xyz="0 0 0.0" rpy="0 0 0" />
-      <geometry>
-        <mesh filename="file://$(find my_robot_description)/meshes/rf_1.STL" />
+        <mesh filename="file://$(find my_robot_description)/meshes/wheelchair_meshes/rf_1.STL" />
+      </geometry>
+      <material name="">
+        <color rgba="0.62745 0.62745 0.62745 1" />
+      </material>
+    </visual>
+    <collision>
+      <origin xyz="0 0 0.0" rpy="0 0 0" />
+      <geometry>
+        <mesh filename="file://$(find my_robot_description)/meshes/wheelchair_meshes/rf_1.STL" />
       </geometry>
     </collision>
@@ -241,14 +241,14 @@
       <origin xyz="0 0 0.0" rpy="0 0 0" />
       <geometry>
-        <mesh filename="file://$(find my_robot_description)/meshes/rb_1.STL" />
-      </geometry>
-      <material name="">
-        <color rgba="0.62745 0.62745 0.62745 1" />
-      </material>
-    </visual>
-    <collision>
-      <origin xyz="0 0 0.0" rpy="0 0 0" />
-      <geometry>
-        <mesh filename="file://$(find my_robot_description)/meshes/rb_1.STL" />
+        <mesh filename="file://$(find my_robot_description)/meshes/wheelchair_meshes/rb_1.STL" />
+      </geometry>
+      <material name="">
+        <color rgba="0.62745 0.62745 0.62745 1" />
+      </material>
+    </visual>
+    <collision>
+      <origin xyz="0 0 0.0" rpy="0 0 0" />
+      <geometry>
+        <mesh filename="file://$(find my_robot_description)/meshes/wheelchair_meshes/rb_1.STL" />
       </geometry>
     </collision>
@@ -269,5 +269,5 @@
       <origin xyz="0 0 0.0" rpy="0 0 0" />
       <geometry>
-        <mesh filename="file://$(find my_robot_description)/meshes/lb_1.STL" />
+        <mesh filename="file://$(find my_robot_description)/meshes/wheelchair_meshes/lb_1.STL" />
       </geometry>
       <material name="">
@@ -278,5 +278,5 @@
       <origin xyz="0 0 0.0" rpy="0 0 0" />
       <geometry>
-        <mesh filename="file://$(find my_robot_description)/meshes/lb_1.STL" />
+        <mesh filename="file://$(find my_robot_description)/meshes/wheelchair_meshes/lb_1.STL" />
       </geometry>
     </collision>
@@ -297,5 +297,5 @@
       <origin xyz="0 0 0" rpy="0 0 0" />
       <geometry>
-        <mesh filename="file://$(find my_robot_description)/meshes/imu_link.STL" />
+        <mesh filename="file://$(find my_robot_description)/meshes/wheelchair_meshes/imu_link.STL" />
       </geometry>
       <material name="">
@@ -306,5 +306,5 @@
       <origin xyz="0 0 0" rpy="0 0 0" />
       <geometry>
-        <mesh filename="file://$(find my_robot_description)/meshes/imu_link.STL" />
+        <mesh filename="file://$(find my_robot_description)/meshes/wheelchair_meshes/imu_link.STL" />
       </geometry>
     </collision>

Commit message: updated URDFs

File: src/my_robot_description/urdf/arm_moveo_urdf.urdf (robot description, URDF)
Before this commit: robot my_robot_description, 15 links, 14 joints
Links:
- link Gripper_Idol_Gear: geometry collision mesh filename=package://my_robot_description/meshes/arm_meshes/Gripper_Id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; visual mesh filename=package://my_robot_description/meshes/arm_meshes/Gripper_Id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
- link Gripper_Servo_Gear: geometry collision mesh filename=package://my_robot_description/meshes/arm_meshes/Gripper_Se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; visual mesh filename=package://my_robot_description/meshes/arm_meshes/Gripper_Se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
- link Pivot_Arm_Gripper_Idol: geometry collision mesh filename=package://my_robot_description/meshes/arm_meshes/Pivot_Arm_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; visual mesh filename=package://my_robot_description/meshes/arm_meshes/Pivot_Arm_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
- link Pivot_Arm_Gripper_Servo: geometry collision mesh filename=package://my_robot_description/meshes/arm_meshes/Pivot_Arm_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; visual mesh filename=package://my_robot_description/meshes/arm_meshes/Pivot_Arm_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
- link Tip_Gripper_Idol: geometry collision mesh filename=package://my_robot_description/meshes/arm_meshes/Tip_Grippe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; visual mesh filename=package://my_robot_description/meshes/arm_meshes/Tip_Grippe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
- link Tip_Gripper_Servo: geometry collision mesh filename=package://my_robot_description/meshes/arm_meshes/Tip_Grippe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; visual mesh filename=package://my_robot_description/meshes/arm_meshes/Tip_Grippe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
- link arm_link: geometry collision mesh filename=package://my_robot_description/meshes/arm_meshes/Link_2_col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; visual mesh filename=package://my_robot_description/meshes/arm_meshes/Link_2.STL
- link base_link: geometry collision mesh filename=package://my_robot_description/meshes/arm_meshes/base_link_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; visual mesh filename=package://my_robot_description/meshes/arm_meshes/base_link.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
- link elbow_link: geometry collision mesh filename=package://my_robot_description/meshes/arm_meshes/Link_3_col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; visual mesh filename=package://my_robot_description/meshes/arm_meshes/Link_3.STL
- link forearm_link: geometry collision mesh filename=package://my_robot_description/meshes/arm_meshes/Link_4_col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; visual mesh filename=package://my_robot_description/meshes/arm_meshes/Link_4.STL
- link shoulder_link: geometry collision mesh filename=package://my_robot_description/meshes/arm_meshes/Link_1_col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; visual mesh filename=package://my_robot_description/meshes/arm_meshes/Link_1.STL
- link wrist_link: geometry collision mesh filename=package://my_robot_description/meshes/arm_meshes/Link_5_col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; visual mesh filename=package://my_robot_description/meshes/arm_meshes/Link_5.STL

File: src/my_robot_description/urdf/my_wheelchair.urdf.xacro (robot description, xacro)
@@ -1,4 +1,7 @@
 <?xml version="1.0"?>
 <robot name="Wheelchair_urdf" xmlns:xacro="http://www.ros.org/wiki/xacro">
+    <xacro:arg name="use_lidar_sim" default="true"/>
+    <xacro:arg name="use_imu_sim" default="true"/>
+    <xacro:arg name="use_mock_hardware" default="false"/>
     <xacro:include filename="common_properties.xacro" />
     <xacro:include filename="wheelchair_base.xacro" />

File: src/my_robot_description/urdf/wheelchair_base.ros2_control.xacro (robot description, xacro)
@@ -1,5 +1,4 @@
 <?xml version="1.0"?>
 <robot xmlns:xacro="http://www.ros.org/wiki/xacro">
-    <xacro:arg name="use_mock_hardware" default="false"/>
     <ros2_control name="MobileBaseHardwareInterface" type="system">
         <hardware>

File: src/my_robot_description/urdf/wheelchair_gazebo.urdf.xacro (robot description, xacro)
@@ -1,5 +1,4 @@
 <?xml version="1.0" encoding="utf-8"?>
 <robot name="Wheelchair_urdf" xmlns:xacro="http://www.ros.org/wiki/xacro">
-    <xacro:arg name="use_lidar_sim" default="true"/>
     <!-- Wheels -->
     <gazebo reference="lb_1">
@@ -62,54 +61,56 @@
     </gazebo>
     <!-- IMU -->
-    <gazebo reference="imu_link">
-        <sensor name="imu" type="imu">
-            <always_on>true</always_on>
-            <update_rate>100</update_rate>
-            <gz_frame_id>imu_link</gz_frame_id>
-            <topic>imu</topic>
-            <imu>
-                <angular_velocity>
-                    <x>
-                        <noise type="gaussian">
-                            <mean>0.0</mean>
-                            <stddev>2e-4</stddev>
-                        </noise>
-                    </x>
-                    <y>
-                        <noise type="gaussian">
-                            <mean>0.0</mean>
-                            <stddev>2e-4</stddev>
-                        </noise>
-                    </y>
-                    <z>
-                        <noise type="gaussian">
-                            <mean>0.0</mean>
-                            <stddev>2e-4</stddev>
-                        </noise>
-                    </z>
-                </angular_velocity>
-                <linear_acceleration>
-                    <x>
-                        <noise type="gaussian">
-                            <mean>0.0</mean>
-                            <stddev>1.7e-2</stddev>
-                        </noise>
-                    </x>
-                    <y>
-                        <noise type="gaussian">
-                            <mean>0.0</mean>
-                            <stddev>1.7e-2</stddev>
-                        </noise>
-                    </y>
-                    <z>
-                        <noise type="gaussian">
-                            <mean>0.0</mean>
-                            <stddev>1.7e-2</stddev>
-                        </noise>
-                    </z>
-                </linear_acceleration>
-            </imu>
-        </sensor>
-    </gazebo>
+    <xacro:if value="$(arg use_imu_sim)">
+        <gazebo reference="imu_link">
+            <sensor name="imu" type="imu">
+                <always_on>true</always_on>
+                <update_rate>100</update_rate>
+                <gz_frame_id>imu_link</gz_frame_id>
+                <topic>imu</topic>
+                <imu>
+                    <angular_velocity>
+                        <x>
+                            <noise type="gaussian">
+                                <mean>0.0</mean>
+                                <stddev>2e-4</stddev>
+                            </noise>
+                        </x>
+                        <y>
+                            <noise type="gaussian">
+                                <mean>0.0</mean>
+                                <stddev>2e-4</stddev>
+                            </noise>
+                        </y>
+                        <z>
+                            <noise type="gaussian">
+                                <mean>0.0</mean>
+                                <stddev>2e-4</stddev>
+                            </noise>
+                        </z>
+                    </angular_velocity>
+                    <linear_acceleration>
+                        <x>
+                            <noise type="gaussian">
+                                <mean>0.0</mean>
+                                <stddev>1.7e-2</stddev>
+                            </noise>
+                        </x>
+                        <y>
+                            <noise type="gaussian">
+                                <mean>0.0</mean>
+                                <stddev>1.7e-2</stddev>
+                            </noise>
+                        </y>
+                        <z>
+                            <noise type="gaussian">
+                                <mean>0.0</mean>
+                                <stddev>1.7e-2</stddev>
+                            </noise>
+                        </z>
+                    </linear_acceleration>
+                </imu>
+            </sensor>
+        </gazebo>
+    </xacro:if>
     <!--Lidar-->
     <xacro:if value="$(arg use_lidar_sim)">
