Commit message: Enable camera support

File: src/my_robot_description/urdf/arm_urdf.xacro (robot description, xacro)
@@ -12,5 +12,5 @@
   </gazebo>
   <xacro:arg name="use_camera" default="false"/>
-  <xacro:include filename="$(find my_robot_description)/sensors/intel_rgbd_cam_d435.urdf.xacro"/>
+  <xacro:include filename="$(find my_robot_description)/sensors/gxivision_lsm36156.urdf.xacro"/>
   <xacro:if value="$(arg use_camera)">
     <!-- Camera Mount Link -->
@@ -18,5 +18,5 @@
       <visual>
         <geometry>
-          <box size="0.05 0.08 0.01"/>
+          <box size="0.05 0.16 0.04"/>
         </geometry>
         <material name="black">
@@ -26,5 +26,5 @@
       <collision>
         <geometry>
-          <box size="0.05 0.08 0.01"/>
+          <box size="0.05 0.16 0.04"/>
         </geometry>
       </collision>
@@ -40,5 +40,8 @@
       <origin xyz="0.05 0 0.025" rpy="0 0 0"/>
     </joint>
-    <xacro:intel_d435 parent="camera_mount" xyz="0 0 0.015" rpy="0 -1.57 3.14"/>
+    <xacro:gxivision_lsm36156
+    parent="camera_mount"
+    xyz="0.018 0 0.02"
+    rpy="0 0 3.14159"/>
   </xacro:if>
 </robot>
