Commit message: modification to URDF

File: src/my_robot_description/urdf/wheelchair_base.xacro (robot description, xacro)
@@ -158,5 +158,5 @@
       <origin xyz="0 0 0" rpy="0 0 0" />
       <geometry>
-        <sphere radius="0.14"/>
+        <mesh filename="file://$(find my_robot_description)/meshes/lf_1.STL" />
       </geometry>
     </collision>
@@ -214,5 +214,5 @@
       <origin xyz="0 0 0" rpy="0 0 0" />
       <geometry>
-        <sphere radius="0.14"/>
+        <mesh filename="file://$(find my_robot_description)/meshes/rf_1.STL" />
       </geometry>
     </collision>
@@ -242,5 +242,5 @@
       <origin xyz="0 0 0" rpy="0 0 0" />
       <geometry>
-        <sphere radius="0.14"/>
+        <mesh filename="file://$(find my_robot_description)/meshes/rb_1.STL" />
       </geometry>
     </collision>
@@ -270,5 +270,5 @@
       <origin xyz="0 0 0" rpy="0 0 0" />
       <geometry>
-        <sphere radius="0.14"/>
+        <mesh filename="file://$(find my_robot_description)/meshes/lb_1.STL" />
       </geometry>
     </collision>

Commit message: Depth camera working and published depth correctly

File: src/my_robot_description/urdf/wheelchair_base.xacro (robot description, xacro)
@@ -310,3 +310,31 @@
     <axis xyz="0 0 0" />
   </joint>
+  <link name="camera_link">
+    <inertial>
+      <origin xyz="0 0 -0.05" rpy="0 0 0" />
+      <mass value="0.035" />
+      <inertia ixx="4.3746E-06" ixy="-1.4987E-22" ixz="-1.9058E-21" iyy="4.3746E-06" iyz="4.5539E-23" izz="4.4197E-06" />
+    </inertial>
+    <visual>
+      <origin xyz="0 0 0" rpy="0 0 0" />
+      <geometry>
+        <box size="0.015 0.130 0.022"/>
+      </geometry>
+      <material name="">
+        <color rgba="0.75294 0.75294 0.75294 1" />
+      </material>
+    </visual>
+    <collision>
+      <origin xyz="0 0 0" rpy="0 0 0" />
+      <geometry>
+        <box size="0.015 0.130 0.022"/>
+      </geometry>
+    </collision>
+  </link>
+  <joint name="camera_joint" type="fixed">
+    <origin xyz="-0.43298 0 0.61687" rpy="0 -0.10674 0" />
+    <parent link="base_link" />
+    <child link="camera_link" />
+    <axis xyz="0 0 0" />
+  </joint>
 </robot>

File: src/my_robot_description/urdf/wheelchair_gazebo.urdf.xacro (robot description, xacro)
@@ -129,15 +129,25 @@
     </gazebo>
     <!-- Camera -->
-    <gazebo reference="lidar_t">
-        <sensor name="depth_camera" type="rgbd_camera">
+    <gazebo reference="camera_link">
+        <sensor name="rgbd_camera" type="rgbd_camera">
             <visualize>True</visualize>
             <baseline>0.2</baseline>
             <pointCloudCutoff>0.5</pointCloudCutoff>
             <pointCloudCutoffMax>3.0</pointCloudCutoffMax>
-            <pose relative_to='lidar_t'>0 0 0 0 0 0</pose>
-            <update_rate>10</update_rate>
-            <always_on>1</always_on>
-            <topic>depth_camera</topic>
-            <gz_frame_id>lidar_t</gz_frame_id>
+            <pose relative_to='camera_link'>0 0 0 0 0 0</pose>
+            <update_rate>5.0</update_rate>
+            <always_on>True</always_on>
+            <topic>rgbd_camera</topic>
+            <gz_frame_id>camera_link</gz_frame_id>
+            <distortionK1>0</distortionK1>
+            <distortionK2>0</distortionK2>
+            <distortionK3>0</distortionK3>
+            <distortionT1>0</distortionT1>
+            <distortionT2>0</distortionT2>
+            <CxPrime>0</CxPrime>
+            <Cx>0</Cx>
+            <Cy>0</Cy>
+            <focalLength>0</focalLength>
+            <hackBaseline>0</hackBaseline>
             <camera>
                 <horizontal_fov>1.047</horizontal_fov>

Commit message: updates

File: src/my_robot_description/urdf/wheelchair_base.xacro (robot description, xacro)
@@ -59,5 +59,5 @@
   </link>
   <joint name="lidar_r_joint" type="fixed">
-    <origin xyz="0.53347 -0.30933 -0.3995" rpy="0 0 0" />
+    <origin xyz="-0.4 -0.30933 0.525" rpy="0 0 -1.5708" />
     <parent link="base_link" />
     <child link="lidar_r" />
@@ -87,5 +87,5 @@
   </link>
   <joint name="lidar_l_joint" type="fixed">
-    <origin xyz="0.53347 0.30688 -0.3995" rpy="0 0 0" />
+    <origin xyz="-0.4 0.30688 0.525" rpy="0 0 1.5708" />
     <parent link="base_link" />
     <child link="lidar_l" />
@@ -311,5 +311,5 @@
   </link>
   <joint name="imu_joint" type="fixed">
-    <origin xyz="0 0 ${base_to_ground_z}" rpy="0 0 0" />
+    <origin xyz="0 0 -0.525" rpy="0 0 0" />
     <parent link="base_link"/>
     <child link="imu_link"/>
