Commit message: updated

File: src/my_robot_description/sensors/intel_rgbd_cam_d435.urdf.xacro (robot description, xacro)
@@ -19,5 +19,5 @@
         <origin xyz="0 0 0" rpy="${M_PI/2} 0.0 ${M_PI/2}"/>
         <geometry>
-          <mesh filename="package://my_robot_description/meshes/d435.stl" />
+          <mesh filename="package://my_robot_description/meshes/arm_meshes/d435.stl" />
         </geometry>
         <material name="black">

File: src/my_robot_description/urdf/arm_urdf.xacro (robot description, xacro)
@@ -13,5 +13,4 @@
   <xacro:arg name="use_camera" default="false"/>
   <xacro:include filename="$(find my_robot_description)/sensors/intel_rgbd_cam_d435.urdf.xacro"/>
-  <!-- Camera macro -->
   <xacro:if value="$(arg use_camera)">
     <!-- Camera Mount Link -->

File: src/my_robot_moveit_config/config/my_robot_description.urdf.xacro (robot description, xacro)
@@ -3,5 +3,5 @@
     <xacro:arg name="initial_positions_file" default="initial_positions.yaml" />
     <!-- Import my_robot_description urdf file -->
-    <xacro:include filename="$(find my_robot_description)/urdf/moveo_urdf.urdf" />
+    <xacro:include filename="$(find my_robot_description)/urdf/arm_moveo_urdf.urdf" />
     <!-- Import control_xacro -->
     <xacro:include filename="my_robot_description.ros2_control.xacro" />
