Commit message: latest

File: src/my_robot_description/urdf/wheelchair/wheelchair.urdf.xacro (robot description, xacro)
@@ -42,7 +42,7 @@
     </visual>
     <collision>
-      <origin xyz="0 0 0" rpy="0 0 0" />
-      <geometry>
-        <mesh filename="package://my_robot_description/meshes/rb_link.STL" />
+      <origin xyz="0 0.0354 0" rpy="1.5708 0 0" />
+      <geometry>
+        <cylinder radius="0.0983" length="0.0306" />
       </geometry>
     </collision>
@@ -70,7 +70,7 @@
     </visual>
     <collision>
-      <origin xyz="0 0 0" rpy="0 0 0" />
-      <geometry>
-        <mesh filename="package://my_robot_description/meshes/lb_link.STL" />
+      <origin xyz="0 -0.0354 0" rpy="1.5708 0 0" />
+      <geometry>
+        <cylinder radius="0.0983" length="0.0306" />
       </geometry>
     </collision>
@@ -84,7 +84,7 @@
   <link name="rcaster_link">
     <inertial>
-      <origin xyz="0.0084911 6.2993E-08 -0.020801" rpy="0 0 0" />
+      <origin xyz="0.0084911 -6.2993E-08 -0.020801" rpy="0 0 0" />
       <mass value="0.066356" />
-      <inertia ixx="0.00015145" ixy="-3.706E-11" ixz="3.0557E-05" iyy="0.00014025" iyz="-3.2899E-11" izz="4.1434E-05" />
+      <inertia ixx="0.00015145" ixy="-3.8993E-11" ixz="3.0557E-05" iyy="0.00014025" iyz="-4.9722E-11" izz="4.1434E-05" />
     </inertial>
     <visual>
@@ -105,14 +105,17 @@
   </link>
   <joint name="rcaster_joint" type="continuous">
-    <origin xyz="-0.2159 -0.31274 0.2032" rpy="0 0 -1.5414" />
+    <origin xyz="-0.2159 -0.31274 0.2032" rpy="0 0 -1.6081" />
     <parent link="base_link" />
     <child link="rcaster_link" />
-    <axis xyz="0 0 -1" />
-  </joint>
+    <axis xyz="0 0 1" />
+    <dynamics damping="0.3" friction="0.0" />
+  </joint>
+  <!-- The exported rcaster_wheel data (mesh, axis, inertia) was corrupted mid-swivel;
+       the right wheel is the same physical part as the left, so reuse the clean left-wheel data. -->
   <link name="rcaster_wheel_link">
     <inertial>
-      <origin xyz="-0.00088601 0.030149 -1.1102E-16" rpy="0 0 0" />
+      <origin xyz="0 -0.030162 0" rpy="0 0 0" />
       <mass value="0.29095" />
-      <inertia ixx="0.00088078" ixy="-2.4602E-05" ixz="-4.4595E-19" iyy="0.0017172" iyz="3.2164E-20" izz="0.00088006" />
+      <inertia ixx="0.00088006" ixy="5.1838E-19" ixz="3.4931E-21" iyy="0.001718" iyz="-4.8105E-20" izz="0.00088006" />
     </inertial>
     <visual>
@@ -126,15 +129,16 @@
     </visual>
     <collision>
-      <origin xyz="0 0 0" rpy="0 0 0" />
-      <geometry>
-        <mesh filename="package://my_robot_description/meshes/rcaster_wheel_link.STL" />
+      <origin xyz="0 -0.030162 0" rpy="1.5708 0 0" />
+      <geometry>
+        <cylinder radius="0.09525" length="0.0539" />
       </geometry>
     </collision>
   </link>
   <joint name="rcaster_wheel_joint" type="continuous">
-    <origin xyz="0.0508 -0.030163 -0.10795" rpy="0 0 -0.029379" />
+    <origin xyz="0.0508 0.030163 -0.10795" rpy="0 0 0" />
     <parent link="rcaster_link" />
     <child link="rcaster_wheel_link" />
-    <axis xyz="0.029375 0.99957 0" />
+    <axis xyz="0 1 0" />
+    <dynamics damping="0.01" friction="0.0" />
   </joint>
   <link name="lcaster_link">
@@ -165,4 +169,5 @@
     <child link="lcaster_link" />
     <axis xyz="0 0 -1" />
+    <dynamics damping="0.3" friction="0.0" />
   </joint>
   <link name="lcaster_wheel_link">
@@ -182,7 +187,7 @@
     </visual>
     <collision>
-      <origin xyz="0 0 0" rpy="0 0 0" />
-      <geometry>
-        <mesh filename="package://my_robot_description/meshes/lcaster_wheel_link.STL" />
+      <origin xyz="0 -0.030162 0" rpy="1.5708 0 0" />
+      <geometry>
+        <cylinder radius="0.09525" length="0.0539" />
       </geometry>
     </collision>
@@ -193,4 +198,5 @@
     <child link="lcaster_wheel_link" />
     <axis xyz="0 1 0" />
+    <dynamics damping="0.01" friction="0.0" />
   </joint>
 </robot>

File: src/my_robot_description/urdf/wheelchair/wheelchair_gazebo.urdf.xacro (robot description, xacro)
@@ -3,7 +3,7 @@
     <!-- Wheels -->
     <gazebo reference="rb_link">
-        <mu1>1000000000000000.0</mu1>
-        <mu2>1000000000000000.0</mu2>
-        <kp>1000000000000.0</kp>
+        <mu1>1.0</mu1>
+        <mu2>1.0</mu2>
+        <kp>1000000.0</kp>
         <kd>10.0</kd>
         <minDepth>0.001</minDepth>
@@ -11,7 +11,7 @@
     </gazebo>
     <gazebo reference="lb_link">
-        <mu1>1000000000000000.0</mu1>
-        <mu2>1000000000000000.0</mu2>
-        <kp>1000000000000.0</kp>
+        <mu1>1.0</mu1>
+        <mu2>1.0</mu2>
+        <kp>1000000.0</kp>
         <kd>10.0</kd>
         <minDepth>0.001</minDepth>
@@ -19,7 +19,7 @@
     </gazebo>
     <gazebo reference="rcaster_link">
-        <mu1>1000000000000000.0</mu1>
-        <mu2>1000000000000000.0</mu2>
-        <kp>1000000000000.0</kp>
+        <mu1>1.0</mu1>
+        <mu2>1.0</mu2>
+        <kp>1000000.0</kp>
         <kd>10.0</kd>
         <minDepth>0.001</minDepth>
@@ -27,7 +27,7 @@
     </gazebo>
     <gazebo reference="rcaster_wheel_link">
-        <mu1>1000000000000000.0</mu1>
-        <mu2>1000000000000000.0</mu2>
-        <kp>1000000000000.0</kp>
+        <mu1>1.0</mu1>
+        <mu2>1.0</mu2>
+        <kp>1000000.0</kp>
         <kd>10.0</kd>
         <minDepth>0.001</minDepth>
@@ -35,18 +35,18 @@
     </gazebo>
     <gazebo reference="lcaster_link">
-        <mu1>1000000000000000.0</mu1>
-        <mu2>1000000000000000.0</mu2>
-        <kp>1000000000000.0</kp>
+        <mu1>1.0</mu1>
+        <mu2>1.0</mu2>
+        <kp>1000000.0</kp>
         <kd>10.0</kd>
         <minDepth>0.001</minDepth>
-        <fdir1>0 0 1</fdir1>
+        <fdir1>1 0 0</fdir1>
     </gazebo>
     <gazebo reference="lcaster_wheel_link">
-        <mu1>1000000000000000.0</mu1>
-        <mu2>1000000000000000.0</mu2>
-        <kp>1000000000000.0</kp>
+        <mu1>1.0</mu1>
+        <mu2>1.0</mu2>
+        <kp>1000000.0</kp>
         <kd>10.0</kd>
         <minDepth>0.001</minDepth>
-        <fdir1>0 0 1</fdir1>
+        <fdir1>1 0 0</fdir1>
     </gazebo>
     <!-- Gazebo Plugins -->
